Commit message: update arm urdf file

File: arm_hand_description/hand_arm/ti5_description/urdf/arm2.urdf (robot description, URDF)
Before this commit: robot arm2, 25 links, 24 joints
Links:
- removed link L_hand_base_link
- removed link L_index_intermediate
- removed link L_index_proximal
- removed link L_index_tip
- removed link L_middle_intermediate
- removed link L_middle_proximal
- removed link L_middle_tip
- removed link L_pinky_intermediate
- removed link L_pinky_proximal
- removed link L_pinky_tip
- removed link L_ring_intermediate
- removed link L_ring_proximal
- removed link L_ring_tip
- removed link L_thumb_distal
- removed link L_thumb_intermediate
- removed link L_thumb_proximal
- removed link L_thumb_proximal_base
- removed link L_thumb_tip
Joints:
- removed joint L_index_intermediate_joint
- removed joint L_index_proximal_joint
- removed joint L_index_tip_joint
- removed joint L_middle_intermediate_joint
- removed joint L_middle_proximal_joint
- removed joint L_middle_tip_joint
- removed joint L_pinky_intermediate_joint
- removed joint L_pinky_proximal_joint
- removed joint L_pinky_tip_joint
- removed joint L_ring_intermediate_joint
- removed joint L_ring_proximal_joint
- removed joint L_ring_tip_joint
- removed joint L_thumb_distal_joint
- removed joint L_thumb_intermediate_joint
- removed joint L_thumb_proximal_pitch_joint
- removed joint L_thumb_proximal_yaw_joint
- removed joint L_thumb_tip_joint
- removed joint fixed_joint
- joint A: limit lower=-3.14 upper=3.14 effort=0 velocity=0 -> lower=-3.14 upper=3.14 effort=80 velocity=2.1750
- joint B: limit lower=-1.9 upper=1.9 effort=0 velocity=0 -> lower=-1.9 upper=1.9 effort=80 velocity=2.1750
- joint C: limit lower=-2.8 upper=2.8 effort=0 velocity=0 -> lower=-2.8 upper=2.8 effort=80 velocity=2.1750
- joint D: limit lower=-3.14 upper=3.14 effort=0 velocity=0 -> lower=-3.14 upper=3.14 effort=80 velocity=2.1750
- joint E: limit lower=-3.14 upper=3.14 effort=0 velocity=0 -> lower=-3.14 upper=3.14 effort=80 velocity=2.1750
- joint F: limit lower=-3.14 upper=3.14 effort=0 velocity=0 -> lower=-3.14 upper=3.14 effort=80 velocity=2.1750
